File: scheme/mine_ver1.sch (KiCad schematic (older format))
At the start: 60 parts, among them IC1 ATMEGA88PA-P, M1 BLDC MOTOR, P1 PROG, P2 I2C, Q1 IRFZ44, Q2 IRFZ44, Q3 IRFZ44, Q4 IRFZ44, Q5 IRFZ44, Q6 IRFZ44, U1 LM2940, U2 74HC08, U3 74HC08, U4 IR2101, U5 IR2101, U6 IR2101, X1 12MHz

Commit message: scheme update & code manipulation
Parts:
- removed C12, C13: 101, symbol CSMALL
- added R23: 3k, symbol R
- C11: value 101 -> 104
Connections:
- wire segments 234 -> 233
Other:
- moved on the sheet: D1, D3, Q1, Q2, Q5, Q6, R10, R11, R12, R13, R17, R18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
